Commit message: fix(kinematics): retune tool length for 22cm gripper (was 24.5cm)
Operator swapped the suction gripper to 22cm on 2026-07-22. Update the
wrist→TCP length consistently across the kinematic model and sim:
  - throwing.py GP8_DIMS tool 0.245 -> 0.220 (wrist→TCP 0.300)
  - robots/gp8.py home EE x 0.705 -> 0.680
  - urdf/gp8_mujoco_suction_tool.xacro tool length
Regenerate warm_db.pkl / warm_db_build_log.json for the new geometry.
Keeping these three in sync avoids the all-pose constant offset that
lands on strike/press height (cf. the 2026-07-21 5mm case).

Co-Authored-By: Claude Opus 4.8 (1M context) <noreply@anthropic.com>

File: urdf/gp8_mujoco_suction_tool.xacro (robot description, xacro)
@@ -5,10 +5,10 @@
     MuJoCo:
       link6 -> gripper body:  (0.080, -0.030, -0.030)
-      gripper -> grip_site:   (0.245, +0.030, +0.030)
-      link6 -> grip_site:     (0.325,  0.000,  0.000)
+      gripper -> grip_site:   (0.220, +0.030, +0.030)
+      link6 -> grip_site:     (0.300,  0.000,  0.000)
     motoman_gp8_support URDF:
       link_6_t -> flange:     (0.080,  0.000,  0.000)
     Therefore:
-      flange -> suction_tool: (0.245,  0.000,  0.000)
+      flange -> suction_tool: (0.220,  0.000,  0.000)
     gp8_control.robots.gp8.forward_kinematics() already returns this TCP/grip_site
     frame, so this URDF is for visualization/frame display only.  Do not add this
@@ -24,7 +24,7 @@
          so the cylinder is centered halfway back toward flange along -X. -->
     <visual name="flange_to_tcp_rod">
-      <origin xyz="-0.1225 0 0" rpy="0 1.57079632679 0"/>
+      <origin xyz="-0.110 0 0" rpy="0 1.57079632679 0"/>
       <geometry>
-        <cylinder radius="0.012" length="0.245"/>
+        <cylinder radius="0.012" length="0.220"/>
       </geometry>
       <material name="suction_tool_red"/>
@@ -39,5 +39,5 @@
   </link>
   <joint name="flange-suction_tool" type="fixed">
-    <origin xyz="0.245 0 0" rpy="0 0 0"/>
+    <origin xyz="0.220 0 0" rpy="0 0 0"/>
     <parent link="flange"/>
     <child link="suction_tool"/>

Commit message: fix(throw): 실측 툴 24cm TCP 반영 — FK 0.700 + GRASP_Z/TRACK_Z −0.02m + URDF/MJCF 동기
2026-08-04 운영자 실측으로 툴 길이 24cm 확정. FK 홈 EE x 0.680→0.700,
flange→suction_tool 0.220→0.240, grip_site 0.245→0.240. 같은 물리 자세를
유지하도록 GRASP_Z 0.062→0.042, TRACK_Z_START/END 0.12/0.05→0.10/0.03
(launch 기본값 미러 포함).

Co-Authored-By: Claude Fable 5 <noreply@anthropic.com>

File: urdf/gp8_mujoco_suction_tool.xacro (robot description, xacro)
@@ -5,10 +5,10 @@
     MuJoCo:
       link6 -> gripper body:  (0.080, -0.030, -0.030)
-      gripper -> grip_site:   (0.220, +0.030, +0.030)
-      link6 -> grip_site:     (0.300,  0.000,  0.000)
+      gripper -> grip_site:   (0.240, +0.030, +0.030)
+      link6 -> grip_site:     (0.320,  0.000,  0.000)
     motoman_gp8_support URDF:
       link_6_t -> flange:     (0.080,  0.000,  0.000)
     Therefore:
-      flange -> suction_tool: (0.220,  0.000,  0.000)
+      flange -> suction_tool: (0.240,  0.000,  0.000)
     gp8_control.robots.gp8.forward_kinematics() already returns this TCP/grip_site
     frame, so this URDF is for visualization/frame display only.  Do not add this
@@ -24,7 +24,7 @@
          so the cylinder is centered halfway back toward flange along -X. -->
     <visual name="flange_to_tcp_rod">
-      <origin xyz="-0.110 0 0" rpy="0 1.57079632679 0"/>
+      <origin xyz="-0.120 0 0" rpy="0 1.57079632679 0"/>
       <geometry>
-        <cylinder radius="0.012" length="0.220"/>
+        <cylinder radius="0.012" length="0.240"/>
       </geometry>
       <material name="suction_tool_red"/>
@@ -39,5 +39,5 @@
   </link>
   <joint name="flange-suction_tool" type="fixed">
-    <origin xyz="0.220 0 0" rpy="0 0 0"/>
+    <origin xyz="0.240 0 0" rpy="0 0 0"/>
     <parent link="flange"/>
     <child link="suction_tool"/>
